File: EAGLE Files/R1.0/OLED Shield.brd (EAGLE design)
At the start: 59.4 x 54.6 mm, 18 parts, among them U1 ARDUINO_SHIELDNOLABELS

Commit message: EAGLE Files
Connections:
- net N$1: no longer PWR.K
- net N$11: now also PWR.K
Routing:
- net N$11: track 37.2 -> 42.3 mm
- net N$1: track 123.1 -> 123.8 mm
Changed lines of the file:
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@@
 <contactref element="OLED1" pad="2"/>
 <contactref element="OLED2" pad="1"/>
-<contactref element="SDCD" pad="A"/>
 <contactref element="R3" pad="P$2"/>
 <contactref element="R1" pad="P$2"/>
-<contactref element="PWR" pad="K"/>
-<wire x1="15.24" y1="30.48" x2="12.7" y2="27.94" width="0.254" layer="16"/>
-<wire x1="20.32" y1="30.48" x2="15.24" y2="30.48" width="0.254" layer="16"/>
-<wire x1="27.94" y1="30.48" x2="30.48" y2="27.94" width="0.254" layer="16"/>
-<wire x1="20.32" y1="30.48" x2="27.94" y2="30.48" width="0.254" layer="16"/>
+<wire x1="27.94" y1="30.48" x2="29.21" y2="29.21" width="0.254" layer="16"/>
+<wire x1="29.21" y1="29.21" x2="30.48" y2="27.94" width="0.254" layer="16"/>
 <wire x1="6.35" y1="68.58" x2="7.62" y2="69.85" width="0.254" layer="1"/>
 <wire x1="6.35" y1="59.69" x2="6.35" y2="68.58" width="0.254" layer="1"/>
@@
 <wire x1="26.67" y1="39.37" x2="26.67" y2="31.75" width="0.254" layer="1"/>
 <via x="48.26" y="72.39" extent="1-16" drill="0.6096"/>
+<contactref element="SDCD" pad="A"/>
+<wire x1="13.97" y1="29.21" x2="12.7" y2="27.94" width="0.254" layer="16"/>
+<wire x1="29.21" y1="29.21" x2="13.97" y2="29.21" width="0.254" layer="16"/>
 </signal>
 <signal name="N$17">
@@
 <wire x1="8.89" y1="35.56" x2="8.6106" y2="36.2712" width="0.254" layer="1"/>
 <wire x1="27.94" y1="35.56" x2="35.56" y2="27.94" width="0.254" layer="16"/>
-<wire x1="8.89" y1="35.56" x2="27.94" y2="35.56" width="0.254" layer="16"/>
+<wire x1="8.89" y1="35.56" x2="20.32" y2="35.56" width="0.254" layer="16"/>
+<wire x1="20.32" y1="35.56" x2="27.94" y2="35.56" width="0.254" layer="16"/>
 <wire x1="8.89" y1="35.56" x2="8.6106" y2="36.2712" width="0.254" layer="16"/>
+<contactref element="PWR" pad="K"/>
+<wire x1="20.32" y1="35.56" x2="20.32" y2="30.48" width="0.254" layer="16"/>
 </signal>
 <signal name="N$12">
